File: forager-pcb/forager-ph.kicad_pcb (KiCad board)
At the start: 2 copper layers, 114.6 x 96.3 mm, 26 parts

Commit message: Partial Heawood Graph Theory diode-free switch wiring done
Parts:
- renumbered BAT to BATTERY
Connections:
- RU1 pad 1: (no net) -> R4 (x2)
- RU1 pad 11: (no net) -> C5 (x2)
- RU1 pad 12: (no net) -> C3 (x2)
- RU1 pad 13: (no net) -> C2 (x2)
- RU1 pad 14: (no net) -> C1 (x2)
- RU1 pad 17: (no net) -> C4 (x2)
- RU1 pad 18: (no net) -> C0 (x2)
- RU1 pad 2: (no net) -> R3 (x2)
- RU1 pad 3: (no net) -> R2 (x2)
- RU1 pad 4: (no net) -> R5 (x2)
- RU1 pad 5: (no net) -> R6 (x2)
- RU1 pad 6: (no net) -> R0 (x2)
- RU1 pad 7: (no net) -> R1 (x2)
- RU1 pad 15: (no net) -> GND
- RU1 pad 16: (no net) -> BAT
- RU1 pad 9: (no net) -> GND
- S3 pad 1: RT2 -> R1
- S3 pad 2: GND -> C2 (x3)
- S3 pad 1: RT4 -> R0
- S3 pad 2: GND -> C4 (x3)
- S3 pad 1: RB4 -> R4
- S3 pad 1: RT0 -> R0
- S3 pad 2: GND -> C0 (x3)
- S3 pad 1: RB0 -> R5
- S3 pad 1: RB3 -> R6
- S3 pad 2: GND -> C3 (x3)
- S3 pad 1: RT1 -> R0
- S3 pad 2: GND -> C1 (x3)
- S3 pad 1: RM1 -> R1
- S3 pad 1: RB1 -> R6
- S3 pad 1: RT3 -> R2
- S3 pad 1: RM4 -> R3
- S3 pad 1: RH1 -> R5
- S3 pad 2: GND -> C5 (x2)
- S3 pad 1: RM0 -> R2
- S3 pad 1: RH0 -> R6
- S3 pad 1: RM3 -> R3
- S3 pad 1: RB2 -> R4
- S3 pad 1: RM2 -> R2
Routing:
- net C5: track 0.00 -> 188.4 mm, vias 0 -> 2
- net C0: track 0.00 -> 186.9 mm, vias 0 -> 3
- net R6: track 0.00 -> 173.9 mm, vias 0 -> 5
- net R5: track 0.00 -> 173.2 mm, vias 0 -> 3
- net R2: track 0.00 -> 168.2 mm, vias 0 -> 5
- net C1: track 0.00 -> 165.2 mm, vias 0 -> 3
- net R4: track 0.00 -> 148.0 mm, vias 0 -> 3
- net C4: track 0.00 -> 133.3 mm, vias 0 -> 3
- net R0: track 0.00 -> 126.3 mm, vias 0 -> 4
- net C2: track 0.00 -> 116.6 mm, vias 0 -> 3
- net C3: track 0.00 -> 101.2 mm, vias 0 -> 4
- net R1: track 0.00 -> 92.6 mm, vias 0 -> 3
- net R3: track 0.00 -> 78.5 mm, vias 0 -> 3
- net GND: track 97.9 -> 143.4 mm, vias 2 -> 8
- net RM4: track 8.41 -> 0.00 mm, vias 1 -> 0
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Other:
- board text added: "BATTERY"
- board text removed: "CLK"
- board text removed: "DIO"
- board text removed: "GND"
- board text removed: "RST"
